File: hardware/RedBoard_Edge.kicad_pcb (KiCad board)
At the start: 2 copper layers, 101.6 x 38.1 mm, 70 parts, among them IC3 LM1117, J1 CONN_025MM, J17 Qwiic_Connector, J18 Qwiic_Connector, J2 ICSP, J3 POWER_JACKSUPER_BOMB_DIGITY, J4 microB, J5 CONN_04, J6 CONN_04, Q1 1A/60V/500mO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

Commit message: conversion to Reds, all parts now point to KiCad library in directory C:/Github
Parts:
- removed G***: LOGO, Custom_Silk:SparkX_Logo
- D5: value Blue -> Green
- R1, R2, R5, R6: value 1k -> 470

Commit message: Conversion to Reds
Parts:
- moved ? 1.80 mm to (119.4, 95.2)
Changed lines of the file:
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@@
     (0 F.Cu signal)
     (31 B.Cu signal)
-    (32 B.Adhes user hide)
-    (33 F.Adhes user hide)
-    (34 B.Paste user hide)
-    (35 F.Paste user hide)
+    (32 B.Adhes user)
+    (33 F.Adhes user)
+    (34 B.Paste user)
+    (35 F.Paste user)
     (36 B.SilkS user)
     (37 F.SilkS user)
-    (38 B.Mask user hide)
+    (38 B.Mask user)
     (39 F.Mask user)
-    (40 Dwgs.User user hide)
+    (40 Dwgs.User user)
     (41 Cmts.User user)
-    (42 Eco1.User user hide)
-    (43 Eco2.User user hide)
+    (42 Eco1.User user)
+    (43 Eco2.User user)
     (44 Edge.Cuts user)
-    (45 Margin user hide)
-    (46 B.CrtYd user hide)
-    (47 F.CrtYd user hide)
-    (48 B.Fab user hide)
+    (45 Margin user)
+    (46 B.CrtYd user)
+    (47 F.CrtYd user)
+    (48 B.Fab user)
     (49 F.Fab user)
   )
@@
     (pad_to_mask_clearance 0.0762)
     (aux_axis_origin 0 0)
-    (visible_elements 7FFE7F1F)
+    (visible_elements 7FFEFF7F)
     (pcbplotparams
       (layerselection 0x010f8_80000001)
@@
   )
   (module Aesthetics:SFE_LOGO_NAME_FLAME_.1 (layer B.Cu)
-    (at 120.65 93.98 180)
+    (at 119.38 95.25 180)
     (descr "SPARKFUN FONT LOGO W/ FLAME - 0.1\" HEIGHT - SILKSCREEN")
     (tags "SPARKFUN FONT LOGO W/ FLAME - 0.1\" HEIGHT - SILKSCREEN")

Commit message: Post Design review changes
Parts:
- removed 5V1, ADC1, GND1: CONN_06SILK_FEMALE_PTH, Connectors:1X06
- removed 5V2, 5V3, GND2, GND3: CONN_04, Connectors:1X04
- removed ?: , Aesthetics:SFE_LOGO_NAME_FLAME_.1
- removed IC3: LM1117, RedBoard:TESTING_SOT223-ALT1
- removed J18: Qwiic_Connector, SparkX:SparkX-1X04_1MM_RA
- removed J3: POWER_JACKSUPER_BOMB_DIGITY, RedBoard:TESTING_POWER_JACK_SMD_OVERPASTE_SUPER_BOMB_DIGITY
- removed JP4, JP6: STAND-OFF, RedBoard:SPARKFUN_STAND-OFF
- removed JP8, JP9: FIDUCIAL1X2, RedBoard:SPARKFUN_FIDUCIAL-1X2
- removed Q3: BSS138, DiscreteSemi:SparkFun-DiscreteSemi-SOT23-3
- removed R10, R8: 4.7k, RedBoard:SPARKFUN-RESISTORS_0603
- removed REF**: Symbol_Barrel_Polarity, Symbols:Symbol_Barrel_Polarity
- removed REF***: OSHW-Logo_7.5x8mm_SilkScreen, Symbols:OSHW-Logo_7.5x8mm_SilkScreen
- removed S1: RESET, NewParts:SWITCH_TACTILE_SPST-NO_0.05A_12V
- added FD1: FIDUCIAL1X2, Aesthetics:FIDUCIAL-MICRO, F.Cu at (160.0, 127.0)
- added FD2: FIDUCIAL1X2, Aesthetics:FIDUCIAL-MICRO, F.Cu at (157.5, 127.0)
- added FD3: FIDUCIAL1X2, Aesthetics:FIDUCIAL-MICRO, F.Cu at (151.5, 121.7)
- added FD4: FIDUCIAL1X2, Aesthetics:FIDUCIAL-MICRO, F.Cu at (156.5, 123.6)
- added H1: STAND-OFF, Hardware:STAND-OFF-TIGHT, F.Cu at (199.4, 114.0)
- added H2: STAND-OFF, Hardware:STAND-OFF-TIGHT, F.Cu at (199.4, 82.3)
- added U6: V_REG_LM1117SOT223, Silicon-Standard:SOT223, F.Cu at (130.2, 99.3)
- C1, C2, C4, C8: value 0.1uF -> 0.1UF-0603-25V-_+80_-20%_; footprint RedBoard:SPARKFUN-CAPACITORS_0603 -> Capacitors:0603
- C10, C9: value 10pF -> 10PF-0603-50V-5%; footprint Capacitors_SMD:C_0603 -> Capacitors:0603
- C11: value 10nF -> 10NF-0603-50V-10%; footprint Capacitors_SMD:C_0603 -> Capacitors:0603
- C12: value 0.1uF -> 0.1UF-0603-25V-_+80_-20%_; footprint Capacitors_SMD:C_0603 -> Capacitors:0603
- C3, C6: value 10uF -> 10UF-POLAR-EIA3216-16V-10%_TANT_; footprint RedBoard:SPARKFUN-CAPACITORS_EIA3216 -> Capacitors:EIA3216
- C5: value 47uF -> 47UF-POLAR-EIA3528-10V-10%; footprint RedBoard:SPARKFUN-CAPACITORS_PANASONIC_D -> Capacitors:EIA3528
- C7: value 1.0uF -> 1.0UF-0603-16V-10%; footprint RedBoard:SPARKFUN-CAPACITORS_0603 -> Capacitors:0603
- D1: value MBRA140 -> DIODE-SHOTTKY_MBRA140; footprint RedBoard:SPARKFUN-DISCRETESEMI_SMA-DIODE -> Silicon-Standard:SMA-DIODE
- D2, D5: value Green -> SPARKFUN-LED_LED-YELLOW-550; footprint NewParts:LED_RED_T1-.75_RT_ANG_PCB -> LED:LED_550_T1-.75_RT_ANG_PCB
- D3: value Yellow -> SPARKFUN-LED_LED-GREEN-550; footprint NewParts:LED_RED_T1-.75_RT_ANG_PCB -> LED:LED_550_T1-.75_RT_ANG_PCB
- D4: value Red -> SPARKFUN-LED_LED-RED-550; footprint NewParts:LED_RED_T1-.75_RT_ANG_PCB -> LED:LED_550_T1-.75_RT_ANG_PCB
- F1: value PTC .5A -> PPTC_HALF-AMP; footprint RedBoard:SPARKFUN-FUSES_1206 -> Fuses:1206
- J17: value Qwiic_Connector -> QWIIC_CONNECTORJS-1MM
- J2: value ICSP -> CONN_03X2SMT
- J4: value microB -> USB_MICRO-B_FEMALE-SMT
- JP1, JP2: value JUMPER-SMT_2_NO_SILK -> JUMPER-SMT_2_NO; footprint Jumpers:SMT-JUMPER_2_NO_SILK -> Jumpers:SMT-JUMPER_2_NO_NO-SILK
- Q1: value 1A/60V/500mO -> MOSFET_PCH-SI2309DS; footprint RedBoard:SPARKFUN-DISCRETESEMI_SOT23-3 -> Silicon-Standard:SOT23-3
- Q2: value BSS138 -> MOSFET-NCH-BSS138; footprint DiscreteSemi:SparkFun-DiscreteSemi-SOT23-3 -> Silicon-Standard:SOT23-3
- R1, R2, R5, R6: value 470 -> 470OHM-0603-1_10W-1%; footprint RedBoard:SPARKFUN-RESISTORS_0603 -> Resistors:0603
- R14: value 715 -> 715OHM-0603-1_10W-1%; footprint RedBoard:SPARKFUN-RESISTORS_0603 -> Resistors:0603
- R15: value 240 -> 240OHM-0603-1_10W-1%; footprint RedBoard:SPARKFUN-RESISTORS_0603 -> Resistors:0603
- R3, R4: value 10k -> 10KOHM-0603-1_10W-1%; footprint RedBoard:SPARKFUN-RESISTORS_0603 -> Resistors:0603
- R7, R9: value 4.7k -> 4.7KOHM-0603-1_10W-1%; footprint RedBoard:SPARKFUN-RESISTORS_0603 -> Resistors:0603
- S2: value SWITCH-SPDT-PTH-11.6X4.0MM -> ROCKER_SWITCH-SPST_PTH_RIGHT_ANGLE; footprint NewParts:RockerSwitch_RA -> Switches:RockerSwitch_RA
- U1: value CH340G -> CH340GSMD; footprint IC:SO16 -> Silicon-Standard:SO16
- U2: value MIC5205 -> V_REG_MIC52053.3V; footprint RedBoard:SPARKFUN-POWERIC_SOT23-5 -> Silicon-Standard:SOT23-5
- U3, U5: footprint NewParts:Standoff_Grounding -> Hardware:STANDOFF_GROUNDING
- U4: footprint RedBoard:SPARKFUN-IC-MICROCONTROLLER_TQFP32-08 -> Silicon-Standard:TQFP32-08
- Y1: value 16MHz -> RESONATOR-16MHZSMD_3.2X1.3; footprint RedBoard:SPARKFUN-CLOCKS_RESONATOR-SMD-3.2X1.3 -> Clocks:RESONATOR-SMD-3.2X1.3
- Y2: value 12MHz -> CRYSTAL-12MHZ
- moved J17 8.12 mm to (138.9, 84.2)
Connections:
- C9 pad 1: Net-(C9-Pad1) -> GND
- C9 pad 2: GND -> Net-(C9-Pad2)
- J4 pad ID: (no net) -> Net-(J4-PadID)
- Q1 pad 1: GND -> Net-(J20-PadP$4)
- R4 pad 1: Net-(J3-PadGND) -> Net-(J20-PadP$4)
- U1 pad 7: Net-(C9-Pad1) -> Net-(C9-Pad2)
- U4 pad 17: /SCK -> Net-(U4-Pad17)
Routing:
- net /HI_SDA: track 38.7 -> 63.4 mm
- net VIN: track 46.0 -> 67.3 mm
- net Net-(C9-Pad2): track 0.00 -> 11.8 mm
- net /HI_SCL: track 45.3 -> 56.8 mm, vias 2 -> 3
- net /RESET: track 37.2 -> 26.0 mm
- net /SCL: track 19.8 -> 8.71 mm, vias 2 -> 0
- net Net-(C9-Pad1): track 9.77 -> 0.00 mm
- net (no net): track 0.03 -> 6.25 mm, vias 0 -> 2
- net /AD7: track 40.1 -> 45.3 mm
- net /AD6: track 39.9 -> 44.9 mm
- net GND: track 20.2 -> 24.3 mm, vias 3 -> 1
- net 3.3V: track 136.2 -> 132.3 mm
- net Net-(J20-PadP$4): track 0.00 -> 2.59 mm
- net 5V: track 216.5 -> 218.1 mm
- net /SCK: track 92.7 -> 91.2 mm
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Other:
- board text added: "A4"
- board text removed: "A6"

Commit message: forgot to save before commit
Parts:
- added LOGO2: OSHW-LOGOS, OSHW-LOGO-S, B.Cu at (109.0, 93.2)
- FD1, FD4: moved to B.Cu
- moved FD2 59.1 mm to (200.7, 86.6)
- moved FD1 57.3 mm to (200.7, 86.6)
- moved FD4 55.1 mm to (104.1, 106.4)
- moved FD3 49.8 mm to (104.1, 106.4)
Routing:
- net /RESET: track 26.0 -> 37.2 mm
- net GND: track 24.3 -> 13.6 mm
Other:
- board text added: "Designed by: Nick Poole"
- board text added: "Revised by: Andy England"
- board text added: "v01"
Changed lines of the file:
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@@
     (area 100.889999 79.172999 202.640001 117.423001)
     (thickness 1.6)
-    (drawings 387)
+    (drawings 390)
     (tracks 562)
     (zones 0)
-    (modules 71)
+    (modules 72)
     (nets 60)
   )
@@
       (net 2 GND))
   )
-  (module Aesthetics:FIDUCIAL-MICRO (layer F.Cu)
-    (at 160.02 127)
+  (module Aesthetics:FIDUCIAL-MICRO (layer B.Cu)
+    (at 200.66 86.614)
     (descr "FIDUCIAL - CIRCLE, 0.25IN")
     (tags "FIDUCIAL - CIRCLE, 0.25IN")
     (attr smd)
-    (fp_text reference FD1 (at 0 0) (layer F.SilkS)
-      (effects (font (thickness 0.15)))
+    (fp_text reference FD1 (at 0 0) (layer B.SilkS)
+      (effects (font (thickness 0.15)) (justify mirror))
     )
-    (fp_text value FIDUCIAL1X2 (at 0 0) (layer F.SilkS)
-      (effects (font (thickness 0.15)))
+    (fp_text value FIDUCIAL1X2 (at 0 0) (layer B.SilkS)
+      (effects (font (thickness 0.15)) (justify mirror))
     )
-    (pad 1 smd circle (at 0 0) (size 0.635 0.635) (layers F.Cu F.Paste F.Mask)
+    (pad 1 smd circle (at 0 0) (size 0.635 0.635) (layers B.Cu B.Paste B.Mask)
       (solder_mask_margin 0.1016))
   )
   (module Aesthetics:FIDUCIAL-MICRO (layer F.Cu)
-    (at 157.48 127)
+    (at 200.66 86.614)
     (descr "FIDUCIAL - CIRCLE, 0.25IN")
     (tags "FIDUCIAL - CIRCLE, 0.25IN")
@@
   )
   (module Aesthetics:FIDUCIAL-MICRO (layer F.Cu)
-    (at 151.511 121.666)
+    (at 104.14 106.426)
     (descr "FIDUCIAL - CIRCLE, 0.25IN")
     (tags "FIDUCIAL - CIRCLE, 0.25IN")
@@
       (solder_mask_margin 0.1016))
   )
-  (module Aesthetics:FIDUCIAL-MICRO (layer F.Cu)
-    (at 156.464 123.571)
+  (module Aesthetics:FIDUCIAL-MICRO (layer B.Cu)
+    (at 104.14 106.426)
     (descr "FIDUCIAL - CIRCLE, 0.25IN")
     (tags "FIDUCIAL - CIRCLE, 0.25IN")
     (attr smd)
-    (fp_text reference FD4 (at 0 0) (layer F.SilkS)
-      (effects (font (thickness 0.15)))
+    (fp_text reference FD4 (at 0 0) (layer B.SilkS)
+      (effects (font (thickness 0.15)) (justify mirror))
     )
-    (fp_text value FIDUCIAL1X2 (at 0 0) (layer F.SilkS)
-      (effects (font (thickness 0.15)))
+    (fp_text value FIDUCIAL1X2 (at 0 0) (layer B.SilkS)
+      (effects (font (thickness 0.15)) (justify mirror))
     )
-    (pad 1 smd circle (at 0 0) (size 0.635 0.635) (layers F.Cu F.Paste F.Mask)
+    (pad 1 smd circle (at 0 0) (size 0.635 0.635) (layers B.Cu B.Paste B.Mask)
       (solder_mask_margin 0.1016))
   )
@@
     (pad NC thru_hole circle (at 3.5 0) (size 1.7 1.7) (drill 1.3) (layers *.Cu *.Mask))
     (pad 2 thru_hole circle (at 2.25 2.5) (size 1.524 1.524) (drill 1) (layers *.Cu *.Mask)
-      (net 2 GND))
+      (net 7 /RESET))
     (pad 1 thru_hole circle (at -2.25 2.5) (size 1.524 1.524) (drill 1) (layers *.Cu *.Mask)
       (net 2 GND))
@@
       (solder_mask_margin 0.1016))
   )
-  (module Aesthetics:SFE_LOGO_NAME_FLAME_.1 (layer B.Cu)
+  (module SFE_LOGO_NAME_FLAME_.1 (layer B.Cu)
     (at 123.444 95.25 180)
     (descr "SPARKFUN FONT LOGO W/ FLAME - 0.1\" HEIGHT - SILKSCREEN")
     (tags "SPARKFUN FONT LOGO W/ FLAME - 0.1\" HEIGHT - SILKSCREEN")
     (attr virtual)
-    (fp_text reference "" (at 0 0 180) (layer B.SilkS)
+    (fp_text reference LOGO1 (at 0 0 180) (layer B.SilkS)
       (effects (font (thickness 0.15)) (justify mirror))
     )
-    (fp_text value "" (at 0 0 180) (layer B.SilkS)
+    (fp_text value SFE_LOGO_NAME_FLAME.1_INCH (at 0 0 180) (layer B.SilkS)
       (effects (font (thickness 0.15)) (justify mirror))
     )
@@
       (xy 8.52932 4.38912) (xy 8.47852 4.52882) (xy 8.40994 4.6482) (xy 8.32866 4.73964)) (layer B.SilkS) (width 0.01))
   )
+  (module OSHW-LOGO-S (layer B.Cu)
+    (at 108.966 93.218 180)
+    (descr "OPEN-SOURCE HARDWARE (OSHW) LOGO - SMALL - SILKSCREEN")
+    (tags "OPEN-SOURCE HARDWARE (OSHW) LOGO - SMALL - SILKSCREEN")
+    (attr virtual)
+    (fp_text reference LOGO2 (at -14.351 -0.846999 450) (layer B.SilkS)
+      (effects (font (thickness 0.15)) (justify mirror))
+    )
+    (fp_text value OSHW-LOGOS (at 0 0 180) (layer B.SilkS)
+      (effects (font (thickness 0.15)) (justify mirror))
+    )
+    (fp_poly (pts (xy 0.3937 -0.9525) (xy 0.5461 -0.87376) (xy 0.92202 -1.1811) (xy 1.1811 -0.92202)
+      (xy 0.87376 -0.5461) (xy 0.9525 -0.3937) (xy 1.0033 -0.23114) (xy 1.48844 -0.18034)
+      (xy 1.48844 0.18034) (xy 1.0033 0.23114) (xy 0.9525 0.3937) (xy 0.87376 0.5461)
+      (xy 1.1811 0.92202) (xy 0.92202 1.1811) (xy 0.5461 0.87376) (xy 0.3937 0.9525)
+      (xy 0.23114 1.0033) (xy 0.18034 1.48844) (xy -0.18034 1.48844) (xy -0.23114 1.0033)
+      (xy -0.3937 0.9525) (xy -0.5461 0.87376) (xy -0.92202 1.1811) (xy -1.1811 0.92202)
+      (xy -0.87376 0.5461) (xy -0.9525 0.3937) (xy -1.0033 0.23114) (xy -1.48844 0.18034)
+      (xy -1.48844 -0.18034) (xy -1.0033 -0.23114) (xy -0.9525 -0.3937) (xy -0.87376 -0.5461)
+      (xy -1.1811 -0.92202) (xy -0.92202 -1.1811) (xy -0.5461 -0.87376) (xy -0.3937 -0.9525)
+      (xy -0.1778 -0.4318) (xy -0.27432 -0.37846) (xy -0.3556 -0.30226) (xy -0.41656 -0.21082)
+      (xy -0.45466 -0.10922) (xy -0.46736 0) (xy -0.45466 0.10922) (xy -0.41402 0.2159)
+      (xy -0.35052 0.30734) (xy -0.2667 0.38354) (xy -0.16764 0.43434) (xy -0.06096 0.46228)
+      (xy 0.0508 0.46482) (xy 0.16002 0.43942) (xy 0.25908 0.38862) (xy 0.34544 0.31496)
+      (xy 0.40894 0.22352) (xy 0.45212 0.11938) (xy 0.46736 0.01016) (xy 0.4572 -0.09906)
+      (xy 0.4191 -0.20574) (xy 0.35814 -0.29972) (xy 0.27686 -0.37592) (xy 0.1778 -0.4318)) (layer B.SilkS) (width 0.01))
+  )
+  (gr_text "Revised by: Andy England" (at 120.142 143.51) (layer Cmts.User)
+    (effects (font (size 1.5 1.5) (thickness 0.3)))
+  )
+  (gr_text "Designed by: Nick Poole" (at 119.38 140.97) (layer Cmts.User)
+    (effects (font (size 1.5 1.5) (thickness 0.3)))
+  )
+  (gr_text v01 (at 195.072 116.078) (layer B.Cu)
+    (effects (font (size 1.5 1.5) (thickness 0.3)) (justify mirror))
+  )
   (gr_text A4 (at 154.432 87.757) (layer F.SilkS)
     (effects (font (size 0.8 0.8) (thickness 0.2)))
@@
   (segment (start 186.26836 92.29236) (end 186.26836 91.44) (width 0.25) (layer F.Cu) (net 1))
   (segment (start 186.055 107.823) (end 186.055 106.299) (width 0.25) (layer F.Cu) (net 2))
-  (segment (start 192.532 114.808) (end 192.532 104.14) (width 0.25) (layer F.Cu) (net 2))
   (segment (start 185.31078 102.7176) (end 185.31078 98.31578) (width 0.25) (layer F.Cu) (net 2))
   (segment (start 185.31078 98.31578) (end 185.293 98.298) (width 0.25) (layer F.Cu) (net 2))
@@
   (segment (start 156.07792 98.298) (end 154.5082 98.298) (width 0.25) (layer F.Cu) (net 6))
   (via (at 154.5082 98.298) (size 0.6) (drill 0.4) (layers F.Cu B.Cu) (net 6))
+  (segment (start 192.532 114.808) (end 192.532 103.6066) (width 0.25) (layer F.Cu) (net 7))
+  (segment (start 192.532 103.6066) (end 195.3006 100.838) (width 0.25) (layer F.Cu) (net 7))
   (segment (start 182.1434 100.457) (end 182.924001 101.237601) (width 0.25) (layer B.Cu) (net 7))
   (segment (start 193.571922 101.237601) (end 193.971523 100.838) (width 0.25) (layer B.Cu) (net 7))
@@
   (segment (start 193.971523 100.838) (end 195.3006 100.838) (width 0.25) (layer B.Cu) (net 7))
   (segment (start 182.1434 98.8314) (end 182.1434 100.457) (width 0.25) (layer B.Cu) (net 7))
-  (segment (start 195.3006 100.838) (end 192.532 103.6066) (width 0.25) (layer F.Cu) (net 7))
   (segment (start 177.292 98.679) (end 177.292 100.584) (width 0.25) (layer F.Cu) (net 7))
   (segment (start 180.62194 98.82378) (end 177.43678 98.82378) (width 0.25) (layer F.Cu) (net 7))

Commit message: QC Double Check Issues
Routing:
- net GND: track 13.6 -> 11.6 mm
Other:
- board text added: "A5"
- board text added: "A6"
Changed lines of the file:
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@@
     (links 179)
     (no_connects 0)
-    (area 100.889999 79.172999 202.640001 117.423001)
+    (area 83.030287 71.214 220.880715 144.86)
     (thickness 1.6)
-    (drawings 390)
-    (tracks 562)
+    (drawings 391)
+    (tracks 560)
     (zones 0)
     (modules 72)
@@
     (trace_min 0.2)
     (segment_width 0.508)
-    (edge_width 0.15)
+    (edge_width 0.24)
     (via_size 0.6)
     (via_drill 0.4)
@@
       (xy 0.4191 -0.20574) (xy 0.35814 -0.29972) (xy 0.27686 -0.37592) (xy 0.1778 -0.4318)) (layer B.SilkS) (width 0.01))
   )
+  (gr_text 3V3 (at 134.62 80.772 90) (layer F.SilkS)
+    (effects (font (size 0.8 0.8) (thickness 0.2)))
+  )
   (gr_text "Revised by: Andy England" (at 120.142 143.51) (layer Cmts.User)
     (effects (font (size 1.5 1.5) (thickness 0.3)))
@@
     (effects (font (size 1.5 1.5) (thickness 0.3)) (justify mirror))
   )
-  (gr_text A4 (at 154.432 87.757) (layer F.SilkS)
+  (gr_text A5 (at 154.432 87.757) (layer F.SilkS)
     (effects (font (size 0.8 0.8) (thickness 0.2)))
   )
-  (gr_text A7 (at 151.892 87.757) (layer F.SilkS)
+  (gr_text A6 (at 151.892 87.757) (layer F.SilkS)
     (effects (font (size 0.8 0.8) (thickness 0.2)))
   )
-  (gr_text A4 (at 151.8285 87.757) (layer B.SilkS)
+  (gr_text A6 (at 151.8285 87.757) (layer B.SilkS)
     (effects (font (size 0.8 0.8) (thickness 0.2)) (justify mirror))
   )
-  (gr_text A4 (at 154.3685 87.757) (layer B.SilkS)
+  (gr_text A5 (at 154.3685 87.757) (layer B.SilkS)
     (effects (font (size 0.8 0.8) (thickness 0.2)) (justify mirror))
   )
@@
   (gr_line (start 120.396 86.614) (end 120.396 88.265) (layer B.SilkS) (width 0.508))
   (gr_line (start 109.347 86.614) (end 120.396 86.614) (layer B.SilkS) (width 0.508))
-  (gr_arc (start 199.39 114.173) (end 202.565 114.173) (angle 90) (layer Edge.Cuts) (width 0.15))
-  (gr_arc (start 199.39 82.423) (end 199.39 79.248) (angle 92.29061004) (layer Edge.Cuts) (width 0.15))
-  (gr_arc (start 104.14 82.423) (end 100.965 82.423) (angle 90) (layer Edge.Cuts) (width 0.15))
-  (gr_arc (start 104.013 114.3) (end 104.013 117.348) (angle 90) (layer Edge.Cuts) (width 0.15))
+  (gr_arc (start 199.39 114.173) (end 202.565 114.173) (angle 90) (layer Edge.Cuts) (width 0.24))
+  (gr_arc (start 199.39 82.423) (end 199.39 79.248) (angle 92.2) (layer Edge.Cuts) (width 0.24))
+  (gr_arc (start 104.14 82.423) (end 100.965 82.423) (angle 90) (layer Edge.Cuts) (width 0.24))
+  (gr_arc (start 104.013 114.3) (end 104.013 117.348) (angle 90) (layer Edge.Cuts) (width 0.24))
   (gr_line (start 177.6476 106.9848) (end 177.6476 108.3564) (layer F.SilkS) (width 0.508))
   (gr_line (start 171.3484 106.9848) (end 171.3484 108.3056) (layer F.SilkS) (width 0.508))
@@
     (effects (font (size 0.8 0.8) (thickness 0.2)))
   )
-  (gr_text QWIIC (at 134.62 81.534 90) (layer F.SilkS)
+  (gr_text QWIIC (at 134.62 84.074 90) (layer F.SilkS)
     (effects (font (size 0.8 0.8) (thickness 0.2)))
   )
@@
     (arrow2b (pts (xy 100.965 73.914) (xy 102.091504 73.327579)))
   )
-  (gr_line (start 100.965 82.423) (end 100.965 114.3) (layer Edge.Cuts) (width 0.15))
-  (gr_line (start 199.39 79.248) (end 104.14 79.248) (layer Edge.Cuts) (width 0.15))
-  (gr_line (start 202.565 114.173) (end 202.565 82.55) (layer Edge.Cuts) (width 0.15))
-  (gr_line (start 104.013 117.348) (end 199.39 117.348) (layer Edge.Cuts) (width 0.15))
+  (gr_line (start 100.965 82.423) (end 100.965 114.3) (layer Edge.Cuts) (width 0.24))
+  (gr_line (start 199.39 79.248) (end 104.14 79.248) (layer Edge.Cuts) (width 0.24))
+  (gr_line (start 202.565 114.173) (end 202.565 82.55) (layer Edge.Cuts) (width 0.24))
+  (gr_line (start 104.013 117.348) (end 199.39 117.348) (layer Edge.Cuts) (width 0.24))
   (dimension 31.75 (width 0.3) (layer Cmts.User)
     (gr_text "1.2500 in" (at 88.566 98.425 270) (layer Cmts.User)
@@
   (segment (start 185.31078 93.24994) (end 186.26836 92.29236) (width 0.25) (layer F.Cu) (net 1))
   (segment (start 186.26836 92.29236) (end 186.26836 91.44) (width 0.25) (layer F.Cu) (net 1))
+  (segment (start 131.84124 112.46612) (end 131.84124 110.50524) (width 0.25) (layer F.Cu) (net 2) (status 400000))
+  (segment (start 131.84124 110.50524) (end 131.826 110.49) (width 0.25) (layer F.Cu) (net 2))
   (segment (start 186.055 107.823) (end 186.055 106.299) (width 0.25) (layer F.Cu) (net 2))
   (segment (start 185.31078 102.7176) (end 185.31078 98.31578) (width 0.25) (layer F.Cu) (net 2))
@@
   (segment (start 183.71312 102.7176) (end 183.71312 103.6026) (width 0.25) (layer F.Cu) (net 2))
   (segment (start 183.71312 103.6026) (end 184.04732 103.9368) (width 0.25) (layer F.Cu) (net 2))
-  (segment (start 131.8514 111.48206) (end 131.7244 111.35506) (width 0.25) (layer F.Cu) (net 2))
-  (segment (start 131.7244 111.35506) (end 131.7244 108.51896) (width 0.25) (layer F.Cu) (net 2))
-  (segment (start 131.84124 112.46612) (end 131.84124 111.49222) (width 0.25) (layer F.Cu) (net 2))
-  (segment (start 131.84124 111.49222) (end 131.8514 111.48206) (width 0.25) (layer F.Cu) (net 2))
   (segment (start 146.558 84.074) (end 146.304 84.074) (width 0.25) (layer F.Cu) (net 3))
   (segment (start 146.304 84.074) (end 144.86636 84.074) (width 0.25) (layer F.Cu) (net 3))
