File: hardware/RedBoard_Edge.sch (KiCad schematic (older format))
At the start: 72 parts, among them J1 CONN_025MM, J17 QWIIC_CONNECTORJS-1MM, J2 CONN_03X2SMT, J20 POWER_JACKSMD, J4 USB_MICRO-B_FEMALE-SMT, J5 CONN_04, J6 CONN_04, Q1 MOSFET_PCH-SI2309DS, Q2 MOSFET-NCH-BSS138, Q3 MOSFET-NCH-BSS138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

Commit message: post design review changes, added switch
Parts:
- removed S2: ROCKER_SWITCH-SPST_PTH_RIGHT_ANGLE, Switches:RockerSwitch_RA, symbol ROCKER_SWITCH-SPST_PTH_RIGHT_ANGLE
- added S2: SWITCH_TOGGLE_SPST_RIGHT_ANGLE, symbol SWITCH_TOGGLE_SPST_RIGHT_ANGLE
Changed lines of the file:
@@
-$EndComp
-$Comp
-L ROCKER_SWITCH-SPST_PTH_RIGHT_ANGLE S2
-U 1 1 59F26123
-P 7150 1600
-F 0 "S2" H 6950 1700 45  0000 L BNN
-F 1 "ROCKER_SWITCH-SPST_PTH_RIGHT_ANGLE" H 6950 1500 45  0000 L BNN
-F 2 "Switches:RockerSwitch_RA" H 7150 1800 20  0001 C CNN
-F 3 "" H 7150 1600 50  0001 C CNN
-F 4 "SWCH-08863" H 7150 1850 60  0000 C CNN "Field4"
-	1    7150 1600
-	-1   0    0    1
 $EndComp
 $Comp
@@
 	7700 3750 7700 3700
 Connection ~ 7700 3700
+$Comp
+L SWITCH_TOGGLE_SPST_RIGHT_ANGLE S2
+U 1 1 5A4D38AF
+P 7150 1600
+F 0 "S2" H 7150 1500 50  0000 C CNN
+F 1 "SWITCH_TOGGLE_SPST_RIGHT_ANGLE" H 7150 1750 50  0000 C CNN
+F 2 "" H 7150 1600 50  0001 C CNN
+F 3 "" H 7150 1600 50  0001 C CNN
+F 4 "PRT-13888" H 7150 1400 50  0001 C CNN "Field4"
+	1    7150 1600
+	1    0    0    -1
+$EndComp
 $EndSCHEMATC
